File: schematic/basic-emulator.kicad_pcb (KiCad board)
At the start: 2 copper layers, 47 x 61.7 mm, 25 parts, among them SW1 SW_SPST

Commit message: feat(schematic): add DAC + high pass for speaker
Parts:
- removed the G*** at (155.8, 100.0)
- removed R2: 500, Resistor_SMD:R_1206_3216Metric_Pad1.30x1.75mm_HandSolder
- removed SW1: SW_SPST, Button_Switch_THT:SW_DIP_SPSTx01_Slide_9.78x4.72mm_W7.62mm_P2.54mm
- added C10: 0.1uF, Capacitor_SMD:C_0603_1608Metric_Pad1.08x0.95mm_HandSolder, B.Cu at (155.6, 84.8)
- added C11: 0.1uF, Capacitor_SMD:C_0603_1608Metric_Pad1.08x0.95mm_HandSolder, B.Cu at (153.6, 96.4)
- added C12: 0.1uF, Capacitor_SMD:C_0603_1608Metric_Pad1.08x0.95mm_HandSolder, B.Cu at (150.6, 91.0)
- added C13: 10nF, Capacitor_SMD:C_0603_1608Metric_Pad1.08x0.95mm_HandSolder, B.Cu at (160.8, 65.6)
- added C14: 10nF, Capacitor_SMD:C_0603_1608Metric_Pad1.08x0.95mm_HandSolder, B.Cu at (160.8, 70.2)
- added C9: 10uF, Capacitor_SMD:C_0603_1608Metric_Pad1.08x0.95mm_HandSolder, B.Cu at (155.6, 83.2)
- added R3: 1kΩ, Resistor_SMD:R_0603_1608Metric_Pad0.98x0.95mm_HandSolder, B.Cu at (158.6, 65.6)
- added R4: 1kΩ, Resistor_SMD:R_0603_1608Metric_Pad0.98x0.95mm_HandSolder, B.Cu at (158.6, 70.2)
- added RV1: 10kΩ, Potentiometer_SMD:Potentiometer_Bourns_3314G_Vertical, B.Cu at (159.6, 76.0)
- added TP1: TestPoint, TestPoint:TestPoint_Pad_D2.0mm, B.Cu at (170.2, 110.0)
- added TP2: TestPoint, TestPoint:TestPoint_Pad_D2.0mm, B.Cu at (176.4, 110.0)
- added U1: PAM8302AAD, Package_SO:SOIC-8_3.9x4.9mm_P1.27mm, B.Cu at (155.6, 91.2)
- moved G*** 1.27 mm to (189.4, 99.8)
Connections:
- A1 pad 2: Net-(A1-GPIO1) -> unconnected-(A1-GPIO1-Pad2)
- A1 pad 4: unconnected-(A1-GPIO2-Pad4) -> SPK_PWM
Routing:
- net /SPK+: track 0.00 -> 46.3 mm, vias 0 -> 2
- net GND: track 213.1 -> 249.5 mm, vias 0 -> 1
- net /SPK-: track 0.00 -> 35.8 mm
- net Net-(C11-Pad1): track 0.00 -> 28.8 mm, vias 0 -> 2
- net +5V: track 174.8 -> 199.1 mm, vias 0 -> 1
- net +3V3: track 27.9 -> 49.5 mm, vias 0 -> 1
- net Net-(A1-GPIO1): track 20.8 -> 0.00 mm
- net SPK_PWM: track 0.00 -> 7.82 mm
- net Net-(C13-Pad1): track 0.00 -> 5.00 mm
- net Net-(U1-IN-): track 0.00 -> 4.63 mm
- net Net-(C14-Pad1): track 0.00 -> 4.43 mm
- net Net-(U1-IN+): track 0.00 -> 2.98 mm
- net unconnected-(A1-GPIO1-Pad2): track 0.00 -> 1.40 mm
- net Net-(D1-DOUT): track 15.0 -> 15.7 mm
Other:
- board text added: "EmuToLife by FDH Systems Revision #1"
- board text removed: "Basic-LD-Emulator by FDH Systems Revision #0"
- board text removed: "ON"
- board text removed: "ON: Xbox OFF: PS3/Wii U"
