File: schematic/basic-emulator.kicad_sch (KiCad schematic)
At the start: 19 parts, among them SW1 SW_SPST

Commit message: feat(schematic): add DAC + high pass for speaker
Parts:
- removed R2: 500, Resistor_SMD:R_1206_3216Metric_Pad1.30x1.75mm_HandSolder, symbol Device:R_US
- removed SW1: SW_SPST, Button_Switch_THT:SW_DIP_SPSTx01_Slide_9.78x4.72mm_W7.62mm_P2.54mm, symbol Switch:SW_SPST
- added C10, C11, C12: 0.1uF, Capacitor_SMD:C_0603_1608Metric_Pad1.08x0.95mm_HandSolder, symbol Device:C
- added C13, C14: 10nF, Capacitor_SMD:C_0603_1608Metric_Pad1.08x0.95mm_HandSolder, symbol Device:C
- added C9: 10uF, Capacitor_SMD:C_0603_1608Metric_Pad1.08x0.95mm_HandSolder, symbol Device:C
- added R3, R4: 1kΩ, Resistor_SMD:R_0603_1608Metric_Pad0.98x0.95mm_HandSolder, symbol Device:R_US
- added RV1: 10kΩ, Potentiometer_SMD:Potentiometer_Bourns_3314G_Vertical, symbol Device:R_Potentiometer_US
- added TP1, TP2: TestPoint, TestPoint:TestPoint_Pad_D2.0mm, symbol Connector:TestPoint
- added U1: PAM8302AAD, Package_SO:SOIC-8_3.9x4.9mm_P1.27mm, symbol Amplifier_Audio:PAM8302AAD
Connections:
- net +3V3: now also U1.1 (~{SD})
- net +5V: now also C10.1, C9.1, U1.6 (VDD)
- net GND: now also C10.2, C12.1, C13.2, C14.2, C9.2, RV1.1, U1.7 (GND)
- net SPK_PWM: now reaches A1.4 (GPIO2)
- net SPK_PWM: now also R3.1
- new net: C13.1, R3.2, R4.1
- new net: C14.1, R4.2, RV1.3
- new net: C11.2, U1.3 (IN+)
- new net: C12.2, U1.4 (IN-)
- new net: C11.1, RV1.2
- new net SPK+: TP1.1, U1.5 (OUT+)
- new net SPK-: TP2.1, U1.8 (OUT-)
Other:
- note added: "Amplifier"
- note added: "RC / Low-Pass"
